File: squares/squares-revB/squares-revB.kicad_sch (KiCad schematic)
At the start: 103 parts, among them J1 USB_C_Pwr, J11 MIX, J12 MUX, J15 Filter, J16 VCA, J2 Inputs, J4 ISP, J7 Sig Out, J8 Line OUT, J9 Line IN, Q1 2N3906, U1 74HC00, U2 40106, U3 74HC00, U4 74HC00, U5 ATtiny2313-20P, U7 MCP602

Commit message: squares: added revB board; added playground firmware
Parts:
- removed Q1: 2N3906, Package_TO_SOT_THT:TO-92_Inline, symbol Transistor_BJT:2N3906
- removed U7: MCP602, Package_DIP:DIP-8_W7.62mm, symbol Device:Opamp_Dual
- added C11: 100n, Capacitor_SMD:C_0805_2012Metric_Pad1.18x1.45mm_HandSolder, symbol Device:C
- added C21, C22, C25, C26: 33n, Capacitor_SMD:C_0805_2012Metric_Pad1.18x1.45mm_HandSolder, symbol Device:C
- added Q1: DMMT5551, DMMT5551:SOIC6_DMMT551_DIO, symbol DMMT5551:DMMT5551-7-F
- added Q2, Q3: 3904, Package_TO_SOT_SMD:SOT-23, symbol Transistor_BJT:MMBT3904
- added Q4: 3906, Package_TO_SOT_SMD:SOT-23, symbol Simulation_SPICE:PNP
- added R1, R4: 220R, Resistor_SMD:R_0805_2012Metric_Pad1.20x1.40mm_HandSolder, symbol Device:R
- added R10, R3, R7: 15k, Resistor_SMD:R_0805_2012Metric_Pad1.20x1.40mm_HandSolder, symbol Device:R
- added R11: 22k, Resistor_SMD:R_0805_2012Metric_Pad1.20x1.40mm_HandSolder, symbol Device:R
- added R12, R9: 4k7, Resistor_SMD:R_0805_2012Metric_Pad1.20x1.40mm_HandSolder, symbol Device:R
- added R55, R56, R62, R64: 470R, Resistor_SMD:R_0805_2012Metric_Pad1.20x1.40mm_HandSolder, symbol Device:R
- added R58: 10k, Resistor_SMD:R_0805_2012Metric_Pad1.20x1.40mm_HandSolder, symbol Device:R
- added U1: MCP6022, Package_DIP:DIP-8_W7.62mm, symbol Device:Opamp_Dual
- C10: renamed from C4; value 100n -> 22p
- C19: renamed from C16; value 10u BP -> 470n; footprint Capacitor_THT:CP_Radial_D5.0mm_P2.00mm -> Capacitor_THT:C_Rect_L7.0mm_W3.5mm_P5.00mm
- C2: renamed from C15; value 10u BP -> 470n; footprint Capacitor_THT:CP_Radial_D5.0mm_P2.00mm -> Capacitor_THT:C_Rect_L7.0mm_W3.5mm_P5.00mm
- D3: value LED -> POWER
- J3: renamed from J2; footprint Connector_PinSocket_2.54mm:PinSocket_2x06_P2.54mm_Vertical -> Connector_PinSocket_2.54mm:PinSocket_2x08_P2.54mm_Vertical
- R20: renamed from R52; value 10k -> 56k
- R31: renamed from R53; value 1k -> 2k7
- U6: value ~ -> MCP6024
- VR1, VR2, VR3, VR4, VR7, VR8: footprint molen:Potentiometer_Alpha_RD901F-40-00D_Single_Vertical_CircularHoles -> Potentiometer_THT:Potentiometer_Alpha_RD901F-40-00D_Single_Vertical
- VR5: renamed from VR6; footprint molen:Potentiometer_Alpha_RD901F-40-00D_Single_Vertical_CircularHoles -> Potentiometer_THT:Potentiometer_Alpha_RD901F-40-00D_Single_Vertical
- VR6: renamed from VR5; footprint molen:Potentiometer_Alpha_RD901F-40-00D_Single_Vertical_CircularHoles -> Potentiometer_THT:Potentiometer_Alpha_RD901F-40-00D_Single_Vertical
- renumbered C12 to C1, C2 to C12, C1 to C13, C3 to C14, C19 to C15, C9 to C16, C14 to C17, C21 to C20, C13 to C23, C20 to C24, C11 to C3, C17 to C4, C6 to C5, C7 to C6, C8 to C7, C5 to C8, C10 to C9, D2 to D1, D1 to D2, J9 to J1, J7 to J10, J1 to J2, J16 to J4, J11 to J5, J15 to J6, J12 to J7, J4 to J9, R46 to R13, R15 to R14, R16 to R15, R8 to R16, R14 to R17, R56 to R18, R57 to R19, R37 to R2, R51 to R21, R55 to R22, R48 to R23, R45 to R24, R54 to R25, R47 to R26, R10 to R27, R50 to R28, R49 to R29, R17 to R30, R9 to R32, R42 to R33, R39 to R34, R44 to R35, R6 to R36, R3 to R37, R23 to R38, R5 to R39, R58 to R40, R24 to R41, R41 to R42, R22 to R43, R4 to R44, R11 to R45, R12 to R46, R19 to R47, R18 to R48, R13 to R49, R38 to R5, R40 to R50, R43 to R51, R35 to R52, R33 to R53, R32 to R54, R34 to R57, R26 to R59, R36 to R6, R28 to R60, R27 to R61, R29 to R63, R30 to R65, R31 to R66, R7 to R8, U4 to U2, U2 to U3, U1 to U4, U3 to U5, U5 to U7
Connections:
- net +5V: now also C11.1, R11.1, R12.1, R58.2, R9.1, U1.8 (V+); no longer J3.13 (Pin_13)
- net AND_a: now also J4.1 (Pin_1); no longer J4.2 (Pin_2)
- net AND_b: now also J4.3 (Pin_3); no longer J4.4 (Pin_4)
- net AND_out: now also J4.5 (Pin_5); no longer J4.6 (Pin_6)
- net CPU_Out_A: now also R66.2; no longer R65.2
- net CPU_Out_B: now also R65.2; no longer R66.2
- net CPU_PWM_0: now also R60.2, C26.2, R62.2; no longer R61.2, U7.14 (PB2)
- net GND: now also J3.3 (Pin_3), C11.2, C21.1, C22.1, C25.1, C26.1, Q2.2 (E), Q3.2 (E), U1.4 (V-); no longer J3.14 (Pin_14), R31.2
- net ISP_nRESET: now also R58.1
- net LINE_In: now also U1.1; no longer U6.7
- net MUX_In_A: no longer U7.7 (PD3)
- net MUX_In_B: no longer U7.8 (PD4)
- net MUX_In_C: no longer U7.9 (PD5)
- net MUX_In_D: now also U5.4; no longer U5.5, U7.11 (PD6)
- net MUX_Out: now also U7.16 (PB4); no longer U7.2 (PD0)
- net MUX_Partial_AB: now also U2.12, U5.8; no longer U2.1, U4.8
- net MUX_Partial_CD: now also U2.2; no longer U2.13
- net MUX_Sel0: now also U4.10, U4.9, U5.5; no longer U4.4, U4.5, U5.4
- net MUX_Sel1: now also U2.1; no longer U2.12
- net REF_2.5v: now also U6.6 (-), U6.7, Q4.2 (B), R1.2, R10.2, R3.1, R4.2; no longer C2.2, U6.5 (+)
- net SqrA_Out: now also U3.12, U7.7 (PD3); no longer U3.2
- net SqrB_Out: now also U3.10, U7.8 (PD4); no longer U3.4
- net SqrC_Out: now also U3.4, U7.9 (PD5); no longer U3.6
- net SqrD_Out: now also U3.2, U7.11 (PD6); no longer U3.8
- net SqrE_Out: now also U3.8; no longer U3.10
- net SqrF_Out: now also U3.6; no longer U3.12
- net VCA_cv: now also J4.4 (Pin_4), R31.1; no longer J4.3 (Pin_3), R20.2
- net VCA_in: now also J4.2 (Pin_2), R20.2; no longer J4.1 (Pin_1)
- net VCA_out: now also J4.6 (Pin_6); no longer J4.5 (Pin_5)
- net at C6.1, VR3.3: now also U3.3; no longer U3.5
- net at R33.1, R42.1: now also U6.5 (+)
- net at R20.1: now also Q1.2, R4.1
- net at R2.2, R5.2: now also U1.2 (-); no longer U6.6 (-)
- net at R26.1: now also U4.5; no longer U5.9
- net at U2.10: now also U2.3; no longer U2.11
- net at U2.9: now also U2.11; no longer U2.3
- net at J3.1 (Pin_1), J3.2 (Pin_2): now also R13.2; no longer R17.1
- net at C5.1, VR2.3: now also U3.11; no longer U3.3
- net at J7.5 (Pin_5), R43.2, R44.2: no longer J7.1 (Pin_1), R36.2, R41.2
- net at J3.11 (Pin_11), J3.12 (Pin_12): now also R30.1; no longer R47.1
- net at U4.11: now also U5.10; no longer U4.10
- net at J3.10 (Pin_10), J3.9 (Pin_9): now also R15.1; no longer R48.1
- net at C8.1, VR1.3: now also U3.13; no longer U3.1
- net at U2.6: now also U2.13; no longer U2.2
- net at R25.2: now also R7.1, U1.7
- net at C16.2, VR6.3: now also U3.9; no longer U3.11
- net at C9.2, VR5.3: now also U3.5; no longer U3.13
- net at J3.15 (Pin_15), J3.16 (Pin_16): now also R47.1; no longer R13.2
- net at J3.5 (Pin_5), J3.6 (Pin_6): now also R17.1; no longer R15.1
- net at J3.7 (Pin_7), J3.8 (Pin_8): now also R14.1; no longer R30.1
- net at R23.1: now also U4.4; no longer U5.10
- net at U4.2, U5.2: now also U4.8; no longer U4.6
- net at U4.3: now also U5.9; no longer U4.9
- net at C7.1, VR4.3: now also U3.1; no longer U3.9
- net at R21.2: now also U4.6; no longer U5.8
- net CPU_PWM_1A: no longer names the net of U7.15 (PB3)
- net CPU_PWM_1A: now also R55.1; no longer R60.2
- net CPU_PWM_1B renamed CPU_Out_C
- net CPU_Out_C: now also U7.2 (PD0); no longer U7.16 (PB4)
- new net: C21.2, R55.2, R56.1
- new net: Q1.1, R7.2, R9.2, U1.6 (-)
- new net: R64.1, U7.14 (PB2)
- new net: Q2.1 (B), Q2.3 (C), Q3.1 (B), Q4.1 (C)
- new net: Q4.3 (E), R31.2
- new net: C25.2, R62.1, R64.2
- new net: J7.1 (Pin_1), R36.2, R41.2
- new net: J3.13 (Pin_13), J3.14 (Pin_14), R48.1
- new net: J3.4 (Pin_4), R11.2
- new net: Q1.3, R1.1
- new net: Q1.4, R10.1, R12.2, U1.5 (+)
- new net: C2.2, R3.2, U1.3 (+)
- new net: Q1.5, Q1.6, Q3.3 (C)
- new net CPU_PWM_1: C22.2, R56.2, R61.2
Other:
- note added: "based on Blue Box VCA by Rene Schmitz"
- moved on the sheet: C19, C2, D1, D2, D3, J1, J4, J5, J8, R13, R14, R15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
